File: kicad/xfactor/xfactor.kicad_sch (KiCad schematic)
At the start: 0 parts

Commit message: Test
Parts:
- added U1: ESP32-S2-WROVER, RF_Module:ESP32-S2-WROVER, symbol RF_Module:ESP32-S2-WROVER
Connections:
- new net: U1.1 (GND), U1.26 (GND), U1.42 (GND), U1.43 (GND)
Changed lines of the file:
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@@
 	(generator_version "9.0")
 	(paper "A4")
+	(symbol
+		(lib_id "RF_Module:ESP32-S2-WROVER")
+		(at 105.41 97.79 0)
+		(unit 1)
+		(exclude_from_sim no)
+		(in_bom yes)
+		(on_board yes)
+		(dnp no)
+		(fields_autoplaced yes)
+		(property "Reference" "U1"
+			(at 107.5533 64.77 0)
+			(effects
+				(font
+					(size 1.27 1.27)
+				)
+				(justify left)
+			)
+		)
+		(property "Value" "ESP32-S2-WROVER"
+			(at 107.5533 67.31 0)
+			(effects
+				(font
+					(size 1.27 1.27)
+				)
+				(justify left)
+			)
+		)
+		(property "Footprint" "RF_Module:ESP32-S2-WROVER"
+			(at 124.46 127 0)
+			(effects
+				(font
+					(size 1.27 1.27)
+				)
+				(hide yes)
+			)
+		)
+		(property "Datasheet" "https://www.espressif.com/sites/default/files/documentation/esp32-s2-wroom_esp32-s2-wroom-i_datasheet_en.pdf"
+			(at 97.79 118.11 0)
+			(effects
+				(font
+					(size 1.27 1.27)
+				)
+				(hide yes)
+			)
+		)
+		(property "Description" "RF Module, ESP32-D0WDQ6 SoC, Wi-Fi 802.11b/g/n, 32-bit, 2.7-3.6V, onboard antenna, SMD"
+			(at 105.41 97.79 0)
+			(effects
+				(font
+					(size 1.27 1.27)
+				)
+				(hide yes)
+			)
+		)
+		(pin "35"
+		)
+		(pin "34"
+		)
+		(pin "33"
+		)
+		(pin "20"
+		)
+		(pin "21"
+		)
+		(pin "2"
+		)
+		(pin "1"
+		)
+		(pin "26"
+		)
+		(pin "42"
+		)
+		(pin "43"
+		)
+		(pin "40"
+		)
+		(pin "39"
+		)
+		(pin "38"
+		)
+		(pin "37"
+		)
+		(pin "36"
+		)
+		(pin "32"
+		)
+		(pin "24"
+		)
+		(pin "22"
+		)
+		(pin "23"
+		)
+		(pin "25"
+		)
+		(pin "27"
+		)
+		(pin "28"
+		)
+		(pin "29"
+		)
+		(pin "30"
+		)
+		(pin "31"
+		)
+		(pin "5"
+		)
+		(pin "4"
+		)
+		(pin "3"
+		)
+		(pin "41"
+		)
+		(pin "6"
+		)
+		(pin "8"
+		)
+		(pin "7"
+		)
+		(pin "9"
+		)
+		(pin "10"
+		)
+		(pin "11"
+		)
+		(pin "12"
+		)
+		(pin "13"
+		)
+		(pin "14"
+		)
+		(pin "15"
+		)
+		(pin "16"
+		)
+		(pin "17"
+		)
+		(pin "18"
+		)
+		(pin "19"
+		)
+		(instances
+			(project ""
+				(path "/dc041239-184b-4404-95d4-5d085ab8623c"
+					(reference "U1")
+					(unit 1)
+				)
+			)
+		)
+	)
 	(sheet_instances
 		(path "/"

Commit message: Test 2
Parts:
- added U2: CDP1802ACEX, Package_DIP:DIP-40_W15.24mm, symbol CPU:CDP1802ACEX
Changed lines of the file:
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@@
 	(paper "A4")
+	(symbol
+		(lib_id "CPU:CDP1802ACEX")
+		(at 191.77 81.28 0)
+		(unit 1)
+		(exclude_from_sim no)
+		(in_bom yes)
+		(on_board yes)
+		(dnp no)
+		(fields_autoplaced yes)
+		(property "Reference" "U2"
+			(at 193.9133 116.84 0)
+			(effects
+				(font
+					(size 1.27 1.27)
+				)
+				(justify left)
+			)
+		)
+		(property "Value" "CDP1802ACEX"
+			(at 193.9133 119.38 0)
+			(effects
+				(font
+					(size 1.27 1.27)
+				)
+				(justify left)
+			)
+		)
+		(property "Footprint" "Package_DIP:DIP-40_W15.24mm"
+			(at 191.77 33.02 0)
+			(effects
+				(font
+					(size 1.27 1.27)
+				)
+				(hide yes)
+			)
+		)
+		(property "Datasheet" "http://www.cosmacelf.com/publications/data-sheets/cdp1802.pdf"
+			(at 191.77 30.48 0)
+			(effects
+				(font
+					(size 1.27 1.27)
+				)
+				(hide yes)
+			)
+		)
+		(property "Description" "8-bit, General Purpose, 5V, 3.2 MHz, Burned-In, DIP-40"
+			(at 191.77 81.28 0)
+			(effects
+				(font
+					(size 1.27 1.27)
+				)
+				(hide yes)
+			)
+		)
+		(pin "25"
+		)
+		(pin "7"
+		)
+		(pin "35"
+		)
+		(pin "19"
+		)
+		(pin "18"
+		)
+		(pin "17"
+		)
+		(pin "33"
+		)
+		(pin "34"
+		)
+		(pin "5"
+		)
+		(pin "6"
+		)
+		(pin "4"
+		)
+		(pin "40"
+		)
+		(pin "20"
+		)
+		(pin "16"
+		)
+		(pin "29"
+		)
+		(pin "28"
+		)
+		(pin "26"
+		)
+		(pin "27"
+		)
+		(pin "30"
+		)
+		(pin "31"
+		)
+		(pin "32"
+		)
+		(pin "9"
+		)
+		(pin "8"
+		)
+		(pin "11"
+		)
+		(pin "10"
+		)
+		(pin "1"
+		)
+		(pin "39"
+		)
+		(pin "38"
+		)
+		(pin "37"
+		)
+		(pin "36"
+		)
+		(pin "24"
+		)
+		(pin "23"
+		)
+		(pin "13"
+		)
+		(pin "12"
+		)
+		(pin "14"
+		)
+		(pin "15"
+		)
+		(pin "2"
+		)
+		(pin "3"
+		)
+		(pin "21"
+		)
+		(pin "22"
+		)
+		(instances
+			(project ""
+				(path "/dc041239-184b-4404-95d4-5d085ab8623c"
+					(reference "U2")
+					(unit 1)
+				)
+			)
+		)
+	)
 	(symbol
 		(lib_id "RF_Module:ESP32-S2-WROVER")

Commit message: Add stuff
Parts:
- added U3: LM319H, Package_TO_SOT_THT:TO-100-10, symbol Comparator:LM319H
Changed lines of the file:
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@@
+	)
+	(symbol
+		(lib_id "Comparator:LM319H")
+		(at 76.2 139.7 0)
+		(unit 1)
+		(exclude_from_sim no)
+		(in_bom yes)
+		(on_board yes)
+		(dnp no)
+		(fields_autoplaced yes)
+		(property "Reference" "U3"
+			(at 76.2 129.54 0)
+			(effects
+				(font
+					(size 1.27 1.27)
+				)
+			)
+		)
+		(property "Value" "LM319H"
+			(at 76.2 132.08 0)
+			(effects
+				(font
+					(size 1.27 1.27)
+				)
+			)
+		)
+		(property "Footprint" "Package_TO_SOT_THT:TO-100-10"
+			(at 76.2 139.7 0)
+			(effects
+				(font
+					(size 1.27 1.27)
+				)
+				(hide yes)
+			)
+		)
+		(property "Datasheet" "http://www.ti.com/lit/ds/symlink/lm319-n.pdf"
+			(at 76.2 139.7 0)
+			(effects
+				(font
+					(size 1.27 1.27)
+				)
+				(hide yes)
+			)
+		)
+		(property "Description" "High Speed Dual Comparator, TO-100-10"
+			(at 76.2 139.7 0)
+			(effects
+				(font
+					(size 1.27 1.27)
+				)
+				(hide yes)
+			)
+		)
+		(pin "6"
+		)
+		(pin "4"
+		)
+		(pin "3"
+		)
+		(pin "2"
+		)
+		(pin "9"
+		)
+		(pin "7"
+		)
+		(pin "8"
+		)
+		(pin "1"
+		)
+		(pin "5"
+		)
+		(pin "10"
+		)
+		(instances
+			(project ""
+				(path "/dc041239-184b-4404-95d4-5d085ab8623c"
+					(reference "U3")
+					(unit 1)
+				)
+			)
+		)
 	)
 	(symbol

Commit message: e23er2re
Parts:
- removed U1: ESP32-S2-WROVER, RF_Module:ESP32-S2-WROVER, symbol RF_Module:ESP32-S2-WROVER
- removed U2: CDP1802ACEX, Package_DIP:DIP-40_W15.24mm, symbol CPU:CDP1802ACEX
- removed U3: LM319H, Package_TO_SOT_THT:TO-100-10, symbol Comparator:LM319H
- added LS1: Speaker, symbol Device:Speaker
- added R1: 1k, Resistor_SMD:R_0805_2012Metric_Pad1.20x1.40mm_HandSolder, symbol Device:R
- added U1: XIAO_ESP32_S3, XIAO_ESP32_S3:MODULE_XIAO_ESP32_S3, symbol XIAO_ESP32_S3:XIAO_ESP32_S3
